File: W1-AT PCB.kicad_sch (KiCad schematic)
At the start: 51 parts, among them J2 Conn_01x05, J3 Conn_01x04, SW1 SW_Push, U1 XC6206PxxxMR, U2 W25Q32JVSS, U3 SRV05-4, U4 RP2040, Y1 12MHz

Commit message: components
Parts:
- removed C1, C2: 22uF, Capacitor_SMD:C_0402_1005Metric, symbol Device:C_Small
- removed Y1: 12MHz, Crystal:Crystal_SMD_3225-4Pin_3.2x2.5mm, symbol Device:Crystal_GND24_Small
- added Y2: CSTNE12M0G520000R0, SnapEDA Library:OSC_CSTNE12M0G520000R0, symbol CSTNE12M0G520000R0:CSTNE12M0G520000R0
- J3: footprint Connector_Molex:Molex_Pico-EZmate_78171-0004_1x04-1MP_P1.20mm_Vertical -> Personalised:Molex_Pico-EZmate_78171-0004_1x04-1MP_P1.20mm_Vertical
- SW1: footprint Button_Switch_SMD:SW_SPST_TL3342 -> Personalised:KXT321LHS
Connections:
- net GND: now also Y2.2
- net XIN: now also Y2.1
- net X_OUT: now also Y2.3
Other:
- moved on the sheet: R1

Commit message: routing
Parts:
- removed U2: W25Q32JVSS, Personalised:W25Q16FWUXIE, symbol Memory_Flash:W25Q32JVSS
- added U5: W25Q32JVSS, Personalised:W25Q16FWUXIE, symbol Memory_Flash:W25Q32JVSS
- R2, R3, R8: value 175Ohm -> 175R
- R4, R5: value 27Ohm -> 27R
- R6: value 10kOhm -> 10K
- R7: value 1kOhm -> 1K
Connections:
- net +3.3V: now also C17.2, U5.8 (VCC); no longer C17.1
- net GND: now also C17.1, U5.4 (GND); no longer C17.2
- net QSPI_SCLK: now also U5.6 (CLK)
- net QSPI_SD0: now also U5.5 (DI(IO0))
- net QSPI_SD1: now also U5.2 (DO(IO1))
- net QSPI_SD2: now also U5.3 (IO2)
- net QSPI_SD3: now also U5.7 (IO3)
- net QSPI_SS: now also U5.1 (~{CS})
- net VBUS renamed VCC
Other:
- moved on the sheet: C17, F2, J3, R1, R7, SW1, U3, Y2
