File: matrix.kicad_sch (KiCad schematic)
At the start: 197 parts, among them SW10 MX_SW_solder, SW11 MX_SW_solder, SW12 ESC, SW13 TAB, SW14 CAPS, SW15 LSFT, SW16 LCTL, SW17 1, SW18 Q, SW19 A, SW2 MX_SW_solder, SW20 ~{LSFT}, SW21 LALT, SW22 2, SW23 W, SW24 S, SW25 Z, SW26 3, SW27 E, SW28 D, SW29 X, SW3 MX_SW_solder, SW30 4, SW31 R, SW32 F, SW33 C, SW34 5, SW35 T, SW36 G, SW37 V, SW38 MX_SW_solder, SW39 6, SW4 MX_SW_solder, SW40 Y, SW41 H, SW42 B, SW43 7, SW44 U, SW45 J, SW46 N, SW47 8, SW48 I, SW49 K, SW5 MX_SW_solder, SW50 M, SW51 9, SW52 O, SW53 L, SW54 <, SW55 0, SW56 P, SW57 :, SW58 >, SW59 -, SW6 MX_SW_solder, SW60 {, SW61 ", SW62 ?, SW63 RALT, SW64 +, SW65 }, SW66 BSPACE, SW67 NLCK, SW68 RSFT, SW69 ~{BSP|\}, SW7 MX_SW_solder, SW70 PIPE, SW71 ENTER, SW72 ~{FN}, SW73 RCTL, SW74 DIVIDE, SW75 N8, SW76 N5, SW77 N2, SW78 SPLIT N-ENTER, SW79 MULT, SW8 MX_SW_solder, SW80 N9, SW81 N6, SW82 N3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

Commit message: changed switch footprint and silkscreen
Parts:
- S1: footprint PCM_Mounting_Keyboard_Stabilizer:Stabilizer_Cherry_MX_2.00u -> PCM_marbastlib-mx:STAB_MX_P_7u
- S3: footprint PCM_Mounting_Keyboard_Stabilizer:Stabilizer_Cherry_MX_7.00u -> PCM_marbastlib-mx:STAB_MX_P_2.25u
- S4, S7, S8, S9: footprint PCM_Mounting_Keyboard_Stabilizer:Stabilizer_Cherry_MX_2.00u -> PCM_marbastlib-mx:STAB_MX_P_2u
- S5: footprint PCM_Mounting_Keyboard_Stabilizer:Stabilizer_Cherry_MX_2.00u -> PCM_marbastlib-mx:STAB_MX_P_2.25u
- S6: footprint PCM_Mounting_Keyboard_Stabilizer:Stabilizer_Cherry_MX_2.00u -> PCM_marbastlib-mx:STAB_MX_P_2.75u
- SW10, SW11, SW12, SW17, SW18, SW19, SW2, SW20, SW22, SW23, SW24, SW25, SW26, SW27, SW28, SW29, SW3, SW30, SW31, SW32, SW33, SW34, SW35, SW36, SW37, SW39, SW4, SW40, SW41, SW42, SW43, SW44, SW45, SW46, SW47, SW48, SW49, SW5, SW50, SW51, SW52, SW53, SW54, SW55, SW56, SW57, SW58, SW59, SW6, SW60, SW61, SW62, SW64, SW65, SW67, SW69, SW7, SW72, SW74, SW75, SW76, SW77, SW78, SW79, SW8, SW80, SW81, SW82, SW83, SW84, SW86, SW88, SW9, SW91, SW93, SW94, SW95, SW96, SW98, SW99: footprint PCM_Switch_Keyboard_Cherry_MX:SW_Cherry_MX_PCB_1.00u -> PCM_marbastlib-mx:SW_MX_1u
- SW13, SW16, SW21, SW63, SW70, SW73: footprint PCM_Switch_Keyboard_Cherry_MX:SW_Cherry_MX_PCB_1.50u -> PCM_marbastlib-mx:SW_MX_1.5u
- SW14, SW92: footprint PCM_Switch_Keyboard_Cherry_MX:SW_Cherry_MX_PCB_1.75u -> PCM_marbastlib-mx:SW_MX_1.75u
- SW15, SW71: footprint PCM_Switch_Keyboard_Cherry_MX:SW_Cherry_MX_PCB_2.25u -> PCM_marbastlib-mx:SW_MX_1u
- SW38: footprint PCM_Switch_Keyboard_Cherry_MX:SW_Cherry_MX_PCB_7.00u -> PCM_marbastlib-mx:SW_MX_1u
- SW66, SW85, SW87, SW97: footprint PCM_Switch_Keyboard_Cherry_MX:SW_Cherry_MX_PCB_2.00u -> PCM_marbastlib-mx:SW_MX_1u
- SW68: footprint PCM_Switch_Keyboard_Cherry_MX:SW_Cherry_MX_PCB_2.75u -> PCM_marbastlib-mx:SW_MX_1u
- SW89, SW90: footprint PCM_Switch_Keyboard_Cherry_MX:SW_Cherry_MX_PCB_1.25u -> PCM_marbastlib-mx:SW_MX_1.25u
